File: mitochondria/conn.kicad_sch (KiCad schematic)
At the start: 0 parts

Commit message: Added 12V DCDC, GPIO connection, related components to library
Parts:
- added J1: ESQ-120-XX-X-D-XX, mc_Footprints:SAMTEC_ESQ-120-XX-X-D-XX, symbol mc_Symbols:ESQ-120-XX-X-D-XX
Connections:
- new net +3.3V: J1.01, J1.17
- new net +5V: J1.02, J1.04
- new net -BATT: J1.06, J1.09, J1.14, J1.20, J1.25, J1.30, J1.34, J1.39
- no-connect marks 0 -> 2
