File: medulla/cond.kicad_sch (KiCad schematic)
At the start: 0 parts

Commit message: 0.1.3-alpha: H-Bridge Completion & I2C Sensor integration
Parts:
- added R17, R18, R19, R20, R8: 10k, symbol Device:R
- added R7: 68k, symbol Device:R
- added TH1: PT1000, symbol Sensor_Temperature:PT1000
- added U5: LM358_DFN, Package_DFN_QFN:DFN-8-1EP_2x2mm_P0.5mm_EP1.05x1.75mm, symbol Amplifier_Operational:LM358_DFN
Connections:
- new net: R18.2, R19.1, R20.1, U5.2 (-)
- new net: R17.2, TH1.1, U5.3 (+)
- new net +3.3V: R17.1, R18.1
- new net +BATT: R7.1
- new net -BATT: R19.2, R8.2, TH1.2
- new net PT1000_Temp: R20.2, U5.1
- new net VBAT_Sense: R7.2, R8.1
