File: medulla/md.kicad_sch (KiCad schematic)
At the start: 0 parts

Commit message: 0.1.3-alpha: H-Bridge Completion & I2C Sensor integration
Parts:
- added C1, C10: 1000n, symbol Device:C_Polarized
- added C11, C12, C2, C3: 470n, symbol Device:C_Polarized
- added C13, C4, C7, C9: 1u, symbol Device:C_Polarized
- added C14, C5, C6, C8: 100u, symbol Device:C_Polarized
- added D1, D10, D11, D14, D15, D16, D17, D2, D20, D3, D4, D9: 1N5819, Diode_THT:D_DO-41_SOD81_P10.16mm_Horizontal, symbol Diode:1N5819
- added D12, D13, D18, D19, D5, D6, D7, D8: 1N4148, Diode_THT:D_DO-35_SOD27_P7.62mm_Horizontal, symbol Diode:1N4148
- added R1, R2, R3, R4, R5, R6, R7, R8: 27, symbol Device:R
- added U1: PCA9685BS, Package_DFN_QFN:QFN-28-1EP_6x6mm_P0.65mm_EP4.25x4.25mm, symbol Driver_LED:PCA9685BS
- added U10, U11, U12, U4, U5, U6, U7, U9: IRF3205STRLPBF, mc_Footprints:SOT3_IRF3205STRLPBF_INF, symbol mc_Symbols:IRF3205STRLPBF
- added U13, U2, U3, U8: IR2104, symbol Driver_FET:IR2104
Connections:
- new net: D12.1 (K), R5.1, U8.7 (HO)
- new net: D12.2 (A), R5.2, U9.1 (G)
- new net: D5.1 (K), R1.1, U2.7 (HO)
- new net: D5.2 (A), R1.2, U4.1 (G)
- new net: D19.1 (K), R8.1, U13.5 (LO)
- new net: D19.2 (A), R8.2, U12.1 (G)
- new net: C9.1, D11.1 (K), U8.8 (VB)
- new net: D7.1 (K), R3.1, U3.7 (HO)
- new net: D7.2 (A), R3.2, U6.1 (G)
- new net: D13.1 (K), R6.1, U8.5 (LO)
- new net: D13.2 (A), R6.2, U10.1 (G)
- new net: D8.1 (K), R4.1, U3.5 (LO)
- new net: C7.1, D10.1 (K), U3.8 (VB)
- new net: C13.1, D20.1 (K), U13.8 (VB)
- new net: C4.1, D9.1 (K), U2.8 (VB)
- new net: D8.2 (A), R4.2, U7.1 (G)
- new net: D6.1 (K), R2.1, U2.5 (LO)
- new net: D6.2 (A), R2.2, U5.1 (G)
- new net: D18.1 (K), R7.1, U13.7 (HO)
- new net: D18.2 (A), R7.2, U11.1 (G)
- new net +12V: C14.2, C5.2, C6.2, C8.2, D10.2 (A), D11.2 (A), D20.2 (A), D9.2 (A), U13.1 (VCC), U2.1 (VCC), U3.1 (VCC), U8.1 (VCC)
- new net +5V: U1.25 (VDD)
- new net +BATT: C1.1, C10.1, C11.1, C12.1, C2.1, C3.1, D1.1 (K), D14.1 (K), D16.1 (K), D3.1 (K), U11.2 (D), U4.2 (D), U6.2 (D), U9.2 (D)
- new net -BATT: C1.2, C10.2, C11.2, C12.2, C14.1, C2.2, C3.2, C5.1, C6.1, C8.1, D15.2 (A), D17.2 (A), D2.2 (A), D4.2 (A), U1.11 (VSS), U1.22 (EXTCLK), U1.29 (VSS), U10.3 (S), U12.3 (S), U13.4 (COM), U2.4 (COM), U3.4 (COM), U5.3 (S), U7.3 (S), U8.4 (COM)
- new net MotA_+: C4.2, D1.2 (A), D2.1 (K), U2.6 (VS), U4.3 (S), U5.2 (D)
- new net MotA_-: C7.2, D3.2 (A), D4.1 (K), U3.6 (VS), U6.3 (S), U7.2 (D)
- new net MotA_D1: U1.4 (LED1), U2.2 (IN)
- new net MotA_D2: U1.5 (LED2), U3.2 (IN)
- new net MotA_Speed: U1.3 (LED0), U2.3 (~{SD}), U3.3 (~{SD})
- new net MotB_+: C9.2, D14.2 (A), D15.1 (K), U10.2 (D), U8.6 (VS), U9.3 (S)
- new net MotB_-: C13.2, D16.2 (A), D17.1 (K), U11.3 (S), U12.2 (D), U13.6 (VS)
- new net MotB_D1: U1.7 (LED4), U8.2 (IN)
- new net MotB_D2: U1.8 (LED5), U13.2 (IN)
- new net MotB_Speed: U1.6 (LED3), U13.3 (~{SD}), U8.3 (~{SD})
- new net SCL: U1.23 (SCL)
- new net SDA: U1.24 (SDA)
