File: medulla/pd.kicad_sch (KiCad schematic)
At the start: 19 parts, among them U1 LM2678S-12

Commit message: 0.1.3-alpha: H-Bridge Completion & I2C Sensor integration
Parts:
- gave numbers to parts that had none: 9
Changed lines of the file:
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@@
 		(dnp no)
 		(fields_autoplaced yes)
-		(property "Reference" "#PWR04"
+		(property "Reference" "#PWR?"
 			(at 29.21 99.06 0)
 			(effects
@@
 				)
 			)
+			(project "medulla"
+				(path "/d5881702-98ec-4aea-8d9c-3c163ba85aa3/e282941a-9b02-493e-88b5-ebcf243042cc"
+					(reference "#PWR?")
+					(unit 1)
+				)
+			)
 		)
 	)
@@
 		(dnp no)
 		(fields_autoplaced yes)
-		(property "Reference" "#PWR02"
+		(property "Reference" "#PWR?"
 			(at 96.52 74.93 0)
 			(effects
@@
 				)
 			)
+			(project "medulla"
+				(path "/d5881702-98ec-4aea-8d9c-3c163ba85aa3/e282941a-9b02-493e-88b5-ebcf243042cc"
+					(reference "#PWR?")
+					(unit 1)
+				)
+			)
 		)
 	)
@@
 		(on_board yes)
 		(dnp no)
-		(property "Reference" "C3"
+		(property "Reference" "C?"
 			(at 42.164 93.98 0)
 			(effects
@@
 				)
 			)
+			(project "medulla"
+				(path "/d5881702-98ec-4aea-8d9c-3c163ba85aa3/e282941a-9b02-493e-88b5-ebcf243042cc"
+					(reference "C?")
+					(unit 1)
+				)
+			)
 		)
 	)
@@
 		(on_board yes)
 		(dnp no)
-		(property "Reference" "C?"
+		(property "Reference" "C7"
 			(at 42.164 30.48 0)
 			(effects
@@
 		(dnp no)
 		(fields_autoplaced yes)
-		(property "Reference" "U1"
+		(property "Reference" "U?"
 			(at 96.52 91.44 0)
 			(effects
@@
 				)
 			)
+			(project "medulla"
+				(path "/d5881702-98ec-4aea-8d9c-3c163ba85aa3/e282941a-9b02-493e-88b5-ebcf243042cc"
+					(reference "U?")
+					(unit 1)
+				)
+			)
 		)
 	)
@@
 		(on_board yes)
 		(dnp no)
-		(property "Reference" "C6"
+		(property "Reference" "C?"
 			(at 144.78 117.348 0)
 			(effects
@@
 				)
 			)
+			(project "medulla"
+				(path "/d5881702-98ec-4aea-8d9c-3c163ba85aa3/e282941a-9b02-493e-88b5-ebcf243042cc"
+					(reference "C?")
+					(unit 1)
+				)
+			)
 		)
 	)
@@
 		(on_board yes)
 		(dnp no)
-		(property "Reference" "C?"
+		(property "Reference" "C12"
 			(at 144.78 53.848 0)
 			(effects
@@
 		(on_board yes)
 		(dnp no)
-		(property "Reference" "C?"
+		(property "Reference" "C9"
 			(at 29.464 30.48 0)
 			(effects
@@
 		(on_board yes)
 		(dnp no)
-		(property "Reference" "C?"
+		(property "Reference" "C10"
 			(at 48.26 30.48 0)
 			(effects
@@
 		(dnp no)
 		(fields_autoplaced yes)
-		(property "Reference" "L1"
+		(property "Reference" "L?"
 			(at 143.51 106.68 90)
 			(effects
@@
 				)
 			)
+			(project "medulla"
+				(path "/d5881702-98ec-4aea-8d9c-3c163ba85aa3/e282941a-9b02-493e-88b5-ebcf243042cc"
+					(reference "L?")
+					(unit 1)
+				)
+			)
 		)
 	)
@@
 		(on_board yes)
 		(dnp no)
-		(property "Reference" "C2"
+		(property "Reference" "C?"
 			(at 35.814 93.98 0)
 			(effects
@@
 				)
 			)
+			(project "medulla"
+				(path "/d5881702-98ec-4aea-8d9c-3c163ba85aa3/e282941a-9b02-493e-88b5-ebcf243042cc"
+					(reference "C?")
+					(unit 1)
+				)
+			)
 		)
 	)
@@
 		(on_board yes)
 		(dnp no)
-		(property "Reference" "C4"
+		(property "Reference" "C?"
 			(at 48.26 93.98 0)
 			(effects
@@
 				)
 			)
+			(project "medulla"
+				(path "/d5881702-98ec-4aea-8d9c-3c163ba85aa3/e282941a-9b02-493e-88b5-ebcf243042cc"
+					(reference "C?")
+					(unit 1)
+				)
+			)
 		)
 	)
@@
 		(on_board yes)
 		(dnp no)
-		(property "Reference" "C5"
+		(property "Reference" "C?"
 			(at 120.65 106.934 90)
 			(effects
@@
 				)
 			)
+			(project "medulla"
+				(path "/d5881702-98ec-4aea-8d9c-3c163ba85aa3/e282941a-9b02-493e-88b5-ebcf243042cc"
+					(reference "C?")
+					(unit 1)
+				)
+			)
 		)
 	)
@@
 		(on_board yes)
 		(dnp no)
-		(property "Reference" "D1"
+		(property "Reference" "D?"
 			(at 131.572 56.896 90)
 			(effects
@@
 				)
 			)
+			(project "medulla"
+				(path "/d5881702-98ec-4aea-8d9c-3c163ba85aa3/e282941a-9b02-493e-88b5-ebcf243042cc"
+					(reference "D?")
+					(unit 1)
+				)
+			)
 		)
 	)
@@
 		(dnp no)
 		(fields_autoplaced yes)
-		(property "Reference" "#PWR05"
+		(property "Reference" "#PWR?"
 			(at 96.52 138.43 0)
 			(effects
@@
 				)
 			)
+			(project "medulla"
+				(path "/d5881702-98ec-4aea-8d9c-3c163ba85aa3/e282941a-9b02-493e-88b5-ebcf243042cc"
+					(reference "#PWR?")
+					(unit 1)
+				)
+			)
 		)
 	)
@@
 		(dnp no)
 		(fields_autoplaced yes)
-		(property "Reference" "#PWR03"
+		(property "Reference" "#PWR?"
 			(at 165.1 48.26 0)
 			(effects
@@
 				)
 			)
+			(project "medulla"
+				(path "/d5881702-98ec-4aea-8d9c-3c163ba85aa3/e282941a-9b02-493e-88b5-ebcf243042cc"
+					(reference "#PWR?")
+					(unit 1)
+				)
+			)
 		)
 	)
@@
 		(dnp no)
 		(fields_autoplaced yes)
-		(property "Reference" "L?"
+		(property "Reference" "L1"
 			(at 143.51 43.18 90)
 			(effects
@@
 		(dnp no)
 		(fields_autoplaced yes)
-		(property "Reference" "#PWR01"
+		(property "Reference" "#PWR?"
 			(at 29.21 35.56 0)
 			(effects
@@
 				)
 			)
+			(project "medulla"
+				(path "/d5881702-98ec-4aea-8d9c-3c163ba85aa3/e282941a-9b02-493e-88b5-ebcf243042cc"
+					(reference "#PWR?")
+					(unit 1)
+				)
+			)
 		)
 	)
@@
 		(on_board yes)
 		(dnp no)
-		(property "Reference" "C?"
+		(property "Reference" "C11"
 			(at 120.65 43.434 90)
 			(effects
@@
 		(on_board yes)
 		(dnp no)
-		(property "Reference" "C?"
+		(property "Reference" "C13"
 			(at 157.48 53.848 0)
 			(effects
@@
 		(dnp no)
 		(fields_autoplaced yes)
-		(property "Reference" "#PWR06"
+		(property "Reference" "#PWR?"
 			(at 165.1 111.76 0)
 			(effects
@@
 				)
 			)
+			(project "medulla"
+				(path "/d5881702-98ec-4aea-8d9c-3c163ba85aa3/e282941a-9b02-493e-88b5-ebcf243042cc"
+					(reference "#PWR?")
+					(unit 1)
+				)
+			)
 		)
 	)
@@
 		(on_board yes)
 		(dnp no)
-		(property "Reference" "D3"
+		(property "Reference" "D?"
 			(at 132.334 116.586 90)
 			(effects
@@
 				)
 			)
+			(project "medulla"
+				(path "/d5881702-98ec-4aea-8d9c-3c163ba85aa3/e282941a-9b02-493e-88b5-ebcf243042cc"
+					(reference "D?")
+					(unit 1)
+				)
+			)
 		)
 	)
@@
 		(on_board yes)
 		(dnp no)
-		(property "Reference" "U?"
+		(property "Reference" "U2"
 			(at 96.52 28.194 0)
 			(effects
@@
 		(on_board yes)
 		(dnp no)
-		(property "Reference" "C1"
+		(property "Reference" "C?"
 			(at 29.464 93.98 0)
 			(effects
@@
 				)
 			)
+			(project "medulla"
+				(path "/d5881702-98ec-4aea-8d9c-3c163ba85aa3/e282941a-9b02-493e-88b5-ebcf243042cc"
+					(reference "C?")
+					(unit 1)
+				)
+			)
 		)
 	)
@@
 		(on_board yes)
 		(dnp no)
-		(property "Reference" "C?"
+		(property "Reference" "C8"
 			(at 35.814 30.48 0)
 			(effects
